File: pcb/fc64x8/fc64x8.sch (EAGLE design)
At the start: 41 parts, among them J1 Micro USB, J2 Outputs, U1 MK20DX128VLF5, U2 AAT3110IGU-5.0-T1, U3 SN74HCT245PWR, X1 16 MHz

Commit message: Draft of Revision B PCB layout
Parts:
- removed C7, C8: 10uF, SparkFun-Passives:CAP_POL1206
- added C12, C13: 10uF, scanlime:C-US0805/NO-OUTLINE
- added JP1, JP2: (no value), pinhead:PINHD-1X1
- C1, C10, C11, C2, C3, C4, C5, C6, C9: device SparkFun-Passives:CAP0603-CAP -> scanlime:C-US0805/NO-OUTLINE
- D1: device SparkFun-LED:LED-YELLOW0603 -> adafruit:LEDCHIP-LED0805
- FB1, FB2: value FB -> FB0805/NO-OUTLINE; device scanlime:FB -> scanlime:FB0805/NO-OUTLINE
- J1: value Micro USB -> (none); device scanlime:USB-FCI-10118194 -> scanlime:USBMINIB
- R1, R10, R11, R2, R3, R4, R5, R6, R7, R8, R9: device SparkFun-Passives:RESISTOR0603-RES -> scanlime:R-US_0805/NO-OUTLINE
Connections:
- net +5V: now also C13.1, FB1.P$2; no longer C7.+, FB1.P$1
- net GND: now also C12.2, C13.2, D1.C, FB2.P$2, J1.GND1, J1.GND2, J1.GND3, J1.GND4, JP1.1, JP2.1; no longer C7.-, C8.-, FB2.P$1, J1.SHIELD@1, J1.SHIELD@2, J1.SHIELD@3, J1.SHIELD@4, J1.SHIELD@5, J1.SHIELD@6, R3.2
- net N$1: now also R3.1; no longer D1.A
- net N$27: now also C12.1; no longer C8.+
- net N$3: now also D1.A, R3.2; no longer D1.C, R3.1
- net N$5: now also FB1.P$1; no longer FB1.P$2
- net N$7: now also FB2.P$1; no longer FB2.P$2
Other:
- note added: "B"
- note removed: "A"
- moved on the sheet: 3.3V, C1, C10, C11, C2, C3, C4, C5, C6, C9, D1, FB1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

Commit message: Update fc64x8 CAD files with final design from Adafruit
- Remove outdated BOM file (Adafruit doesn't use a separate BOM spreadsheet)
- Added fiducials
- Added Adafruit logo
Parts:
- added FID1, FID2, FID3: FIDUCIAL"", microbuilder:FIDUCIAL""
- C1, C5: value 2.2uF -> 10uF
- R10, R11, R4, R5, R6, R7, R8, R9: value 75 -> 68
Changed lines of the file:
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@@
 <?xml version="1.0" encoding="utf-8"?>
 <!DOCTYPE eagle SYSTEM "eagle.dtd">
-<eagle version="6.5.0">
+<eagle version="6.3">
 <drawing>
 <settings>
@@
 <part name="GND1" library="supply1" deviceset="GND" device=""/>
 <part name="U1" library="scanlime" deviceset="MK20DX128VLF5" device="" value="MK20DX128VLF5"/>
-<part name="C1" library="scanlime" deviceset="C-US" device="0805/NO-OUTLINE" value="2.2uF"/>
+<part name="C1" library="scanlime" deviceset="C-US" device="0805/NO-OUTLINE" value="10uF"/>
 <part name="C2" library="scanlime" deviceset="C-US" device="0805/NO-OUTLINE" value="0.1uF"/>
 <part name="C3" library="scanlime" deviceset="C-US" device="0805/NO-OUTLINE" value="0.1uF"/>
 <part name="C4" library="scanlime" deviceset="C-US" device="0805/NO-OUTLINE" value="0.1uF"/>
-<part name="C5" library="scanlime" deviceset="C-US" device="0805/NO-OUTLINE" value="2.2uF"/>
+<part name="C5" library="scanlime" deviceset="C-US" device="0805/NO-OUTLINE" value="10uF"/>
 <part name="C6" library="scanlime" deviceset="C-US" device="0805/NO-OUTLINE" value="0.1uF"/>
 <part name="FB1" library="scanlime" deviceset="FB" device="0805/NO-OUTLINE"/>
@@
 <part name="C10" library="scanlime" deviceset="C-US" device="0805/NO-OUTLINE" value="2.2uF"/>
 <part name="C11" library="scanlime" deviceset="C-US" device="0805/NO-OUTLINE" value="0.1uF"/>
-<part name="R4" library="scanlime" deviceset="R-US_" device="0805/NO-OUTLINE" value="75"/>
-<part name="R5" library="scanlime" deviceset="R-US_" device="0805/NO-OUTLINE" value="75"/>
-<part name="R6" library="scanlime" deviceset="R-US_" device="0805/NO-OUTLINE" value="75"/>
-<part name="R7" library="scanlime" deviceset="R-US_" device="0805/NO-OUTLINE" value="75"/>
-<part name="R8" library="scanlime" deviceset="R-US_" device="0805/NO-OUTLINE" value="75"/>
-<part name="R9" library="scanlime" deviceset="R-US_" device="0805/NO-OUTLINE" value="75"/>
-<part name="R10" library="scanlime" deviceset="R-US_" device="0805/NO-OUTLINE" value="75"/>
-<part name="R11" library="scanlime" deviceset="R-US_" device="0805/NO-OUTLINE" value="75"/>
+<part name="R4" library="scanlime" deviceset="R-US_" device="0805/NO-OUTLINE" value="68"/>
+<part name="R5" library="scanlime" deviceset="R-US_" device="0805/NO-OUTLINE" value="68"/>
+<part name="R6" library="scanlime" deviceset="R-US_" device="0805/NO-OUTLINE" value="68"/>
+<part name="R7" library="scanlime" deviceset="R-US_" device="0805/NO-OUTLINE" value="68"/>
+<part name="R8" library="scanlime" deviceset="R-US_" device="0805/NO-OUTLINE" value="68"/>
+<part name="R9" library="scanlime" deviceset="R-US_" device="0805/NO-OUTLINE" value="68"/>
+<part name="R10" library="scanlime" deviceset="R-US_" device="0805/NO-OUTLINE" value="68"/>
+<part name="R11" library="scanlime" deviceset="R-US_" device="0805/NO-OUTLINE" value="68"/>
 <part name="J2" library="pinhead" deviceset="PINHD-2X8" device="" value="Outputs"/>
 <part name="GND10" library="supply1" deviceset="GND" device=""/>
@@
 <part name="JP2" library="pinhead" deviceset="PINHD-1X1" device=""/>
 <part name="GND11" library="supply1" deviceset="GND" device=""/>
+<part name="FID1" library="microbuilder" deviceset="FIDUCIAL" device="&quot;&quot;"/>
+<part name="FID2" library="microbuilder" deviceset="FIDUCIAL" device="&quot;&quot;"/>
+<part name="FID3" library="microbuilder" deviceset="FIDUCIAL" device="&quot;&quot;"/>
 </parts>
 <sheets>
@@
 <instance part="JP2" gate="G$1" x="226.06" y="147.32"/>
 <instance part="GND11" gate="1" x="213.36" y="139.7"/>
+<instance part="FID1" gate="G$1" x="7.62" y="170.18"/>
+<instance part="FID2" gate="G$1" x="7.62" y="162.56"/>
+<instance part="FID3" gate="G$1" x="12.7" y="167.64"/>
 </instances>
 <busses>
